File: hardware/JAMMA2Console.sch (KiCad schematic (older format))
At the start: 16 parts

Commit message: Just updating on how things are going. Its pretty messy at the moment, but in the same time I'm not even close to finishing the schematic. I'm going to split up the schematic into different pages for audio, video and digital to make things cleaner (and which hasn't even been started yet).
Parts:
- removed J?: Conn_02x28_Top_Bottom, symbol Connector_Generic:Conn_02x28_Top_Bottom
- removed J? (x2): DB15_Female, symbol Connector:DB15_Female
- removed RN? (x5): 100R, symbol Device:R_Pack04
- removed U? (x2): 74LVC4245, Package_SO:TSSOP-24_4.4x7.8mm_P0.65mm, symbol Logic_LevelTranslator:SN74AVC8T245PW
- removed U?: STM32F030C8Tx, Package_QFP:LQFP-48_7x7mm_P0.5mm, symbol MCU_ST_STM32F0:STM32F030C8Tx
- added C1: 510p, Capacitor_SMD:C_0603_1608Metric, symbol Device:C
- added C10, C11, C13, C14, C15, C16, C17, C18, C19, C2, C20, C21, C3, C4, C6, C7, C8, C9: 100n, Capacitor_SMD:C_0603_1608Metric, symbol Device:C
- added C12, C5: 10u, Capacitor_SMD:C_0603_1608Metric, symbol Device:C
- added C22, C23: 10u, Capacitor_SMD:C_0805_2012Metric, symbol Device:C
- added J1: Conn_02x28_JAMMA, Console2JAMMA:JAMMA_56_2x28_P3.96mm, symbol Console2JAMMA:Conn_02x28_JAMMA
- added J5, J6: DB15_Female, Connector_Dsub:DSUB-15_Male_Horizontal_P2.77x2.84mm_EdgePinOffset14.56mm_Housed_MountingHolesOffset15.98mm, symbol Connector:DB15_Female
- added J7: DF1BZ-34DP-2.5DSA, Connector_PinHeader_2.54mm:PinHeader_2x17_P2.54mm_Vertical, symbol Connector_Generic:Conn_02x17_Odd_Even
- added R1: 620, Resistor_SMD:R_0603_1608Metric, symbol Device:R
- added R10, R6, R7, R9: 100K, Resistor_SMD:R_0603_1608Metric, symbol Device:R
- added R2: 680k, Resistor_SMD:R_0603_1608Metric, symbol Device:R
- added R3, R4, R5: 10k, Resistor_SMD:R_0603_1608Metric, symbol Device:R
- added R8: 47K, Resistor_SMD:R_0603_1608Metric, symbol Device:R
- added R?: 10K, Resistor_SMD:R_0603_1608Metric, symbol Device:R
- added RN10, RN11, RN12, RN13, RN14, RN15, RN16, RN17, RN18, RN19, RN20, RN21, RN7, RN8, RN9: 10k, Resistor_SMD:R_Array_Convex_4x0603, symbol Device:R_Pack04
- added RN? (x5): 4K7, Resistor_SMD:R_Array_Concave_4x0603, symbol Device:R_Pack04
- added U1: STM32F103V8Tx, Package_QFP:LQFP-100_14x14mm_P0.5mm, symbol MCU_ST_STM32F1:STM32F103V8Tx
- added U3, U4: 74LVC4245, Package_SO:TSSOP-24_4.4x7.8mm_P0.65mm, symbol Logic_LevelTranslator:SN74AVC8T245PW
- added U5: LM1881, Package_SO:SOIC-8_3.9x4.9mm_P1.27mm, symbol Video:LM1881
- added U6: TL072, Package_SO:SOIC-8_3.9x4.9mm_P1.27mm, symbol Amplifier_Operational:TL072
- J2: renamed from J?; footprint (none) -> Console2JAMMA:Conn_SCART_Female
- J3: renamed from J?; footprint (none) -> Connector_Dsub:DSUB-15-HD_Female_Horizontal_P2.29x1.98mm_EdgePinOffset8.35mm_Housed_MountingHolesOffset10.89mm
- J4: renamed from J?; footprint (none) -> Console2JAMMA:RCA_Switchchraft_Dual
- RN3: renamed from RN?; value 100R -> 4K7; footprint (none) -> Resistor_SMD:R_Array_Concave_4x0603
- gave numbers to parts that had none: 1
Connections:
- net labels added: -12V, Audio_Mono, P1&P2_Shifter_DIR, P1P2_Shifter_DIR, P1_Button1, P1_Button10, P1_Button11, P1_Button12, P1_Button2, P1_Button3, P1_Button4, P1_Button5, P1_Button6, P1_Button7, P1_Button8, P1_Button9, P1_HK, P1_LK, P1_MK, P1_Shifter_DIR, P2_Button1, P2_Button10, P2_Button11, P2_Button12, P2_Button2, P2_Button3, P2_Button4, P2_Button5, P2_Button6, P2_Button7, P2_Button8, P2_Button9, P2_HK, P2_LK, P2_MK, P2_Shifter_DIR, SCART_Audio_L, SCART_Audio_R, SCART_Blue, SCART_COMP, SCART_CSYNC, SCART_Green, SCART_Red, VGA_Blue, VGA_Green, VGA_HSYNC, VGA_Red, VGA_SCK, VGA_SDA, VGA_VSYNC
- net labels removed: CYSNC, PA0, PA1, PA10, PA11, PA12, PA13, PA14, PA15, PA2, PA3, PA4, PA5, PA6, PA7, PA8, PA9, PB0, PB1, PB10, PB11, PB12, PB13, PB14, PB15, PB2, PB3, PB4, PB5, PB6, PB7, PB8, PB9
- wire segments 224 -> 498
- no-connect marks 16 -> 46
Other:
- note added: "3V3 I/O to and from Level Shifter"
- note added: "5V Button Inputs from \nArcade Machine"
- note added: "Audio in"
- note added: "CPS2 Style Kick Harness"
- note added: "Controller Ports & Level Conversion"
- note added: "JAMMA Connector"
- note added: "Microcontroller"
- note added: "Player 1"
- note added: "Player 2"
- note added: "Slew Rate Control"
- note added: "Stereo to Mono Combiner"
- note added: "Sync Stripper"
- note added: "TO DO LIST:\n- pam8106 audio amp + audio controls\n- BA7046F/LM1881 for Composite Sync\n- Audio mono combiner circuit\n- Potentiometers for video signal\n- VGA input option (dreamcasts etc.)\n - Also for Dreamcast, and Sync combiner will be necessary\n- THS7375 video amp\n- Button Remapping for software"
- note added: "VGA in"
- note added: "Video & Audio IN"
- note removed: ""JAMMA" Connector"
- note removed: "Slew Rate Control Resistors"
- note removed: "TO DO LIST:\n- pam8106 audio amp + audio controls\n- BA7406 for Composite Sync\n- Audio mono combiner circuit\n- Potentiometers for video signal\n- VGA input option (dreamcasts etc.)\n - Also for Dreamcast, and Sync combiner will be necessary\n- THS7375 video amp\n- Button Remapping for software"
- moved on the sheet: J2, J3, J4, J6, RN3

Commit message: More work on various schematic files, added footprint for the speaker out terminal connectors.
Parts:
- removed C1: 510p, Capacitor_SMD:C_0603_1608Metric, symbol Device:C
- removed C10, C11, C13, C14, C15, C16, C17, C18, C19, C2, C20, C21, C3, C4, C6, C7, C8, C9: 100n, Capacitor_SMD:C_0603_1608Metric, symbol Device:C
- removed C12, C5: 10u, Capacitor_SMD:C_0603_1608Metric, symbol Device:C
- removed C22, C23: 10u, Capacitor_SMD:C_0805_2012Metric, symbol Device:C
- removed J4: Conn_Coaxial_x2, Console2JAMMA:RCA_Switchchraft_Dual, symbol Connector:Conn_Coaxial_x2
- removed J5: DB15_Female, Connector_Dsub:DSUB-15_Male_Horizontal_P2.77x2.84mm_EdgePinOffset14.56mm_Housed_MountingHolesOffset15.98mm, symbol Connector:DB15_Female
- removed J7: DF1BZ-34DP-2.5DSA, Connector_PinHeader_2.54mm:PinHeader_2x17_P2.54mm_Vertical, symbol Connector_Generic:Conn_02x17_Odd_Even
- removed R1: 620, Resistor_SMD:R_0603_1608Metric, symbol Device:R
- removed R10, R6, R7, R9: 100K, Resistor_SMD:R_0603_1608Metric, symbol Device:R
- removed R2: 680k, Resistor_SMD:R_0603_1608Metric, symbol Device:R
- removed R3, R4, R5: 10k, Resistor_SMD:R_0603_1608Metric, symbol Device:R
- removed R8: 47K, Resistor_SMD:R_0603_1608Metric, symbol Device:R
- removed R?: 10K, Resistor_SMD:R_0603_1608Metric, symbol Device:R
- removed RN10, RN11, RN12, RN13, RN14, RN15, RN16, RN17, RN7, RN8, RN9: 10k, Resistor_SMD:R_Array_Convex_4x0603, symbol Device:R_Pack04
- removed RN3, RN? (x5): 4K7, Resistor_SMD:R_Array_Concave_4x0603, symbol Device:R_Pack04
- removed U1: STM32F103V8Tx, Package_QFP:LQFP-100_14x14mm_P0.5mm, symbol MCU_ST_STM32F1:STM32F103V8Tx
- removed U2, U3, U4: 74LVC4245, Package_SO:TSSOP-24_4.4x7.8mm_P0.65mm, symbol Logic_LevelTranslator:SN74AVC8T245PW
- removed U5: LM1881, Package_SO:SOIC-8_3.9x4.9mm_P1.27mm, symbol Video:LM1881
- removed U6: TL072, Package_SO:SOIC-8_3.9x4.9mm_P1.27mm, symbol Amplifier_Operational:TL072
- added D1, D10, D12, D13, D14, D2, D3, D4, D5, D6, D7, D8, D9: LESD3Z5.0CMT1G, Diode_SMD:D_SOD-323, symbol Console2JAMMA:D_TVS_ALT_45deg
- added J4: DF1BZ-34DP-2.5DSA, Connector_PinHeader_2.54mm:PinHeader_2x17_P2.54mm_Vertical, symbol Connector_Generic:Conn_02x17_Odd_Even
- added J5: Conn_Coaxial_x2, Console2JAMMA:RCA_Switchchraft_Dual, symbol Connector:Conn_Coaxial_x2
- added J7: DB15_Female, Connector_Dsub:DSUB-15_Female_Horizontal_P2.77x2.84mm_EdgePinOffset7.70mm_Housed_MountingHolesOffset9.12mm, symbol Connector:DB15_Female
- added J8: Conn_01x04, Console2JAMMA:PhoenixContact_PTS_1,5_4-5_1x4_P5.00mm_Horizontal, symbol Connector_Generic:Conn_01x04
- added RN22, RN23: 4K7, Resistor_SMD:R_Array_Convex_4x0603, symbol Device:R_Pack04
- J6: footprint Connector_Dsub:DSUB-15_Male_Horizontal_P2.77x2.84mm_EdgePinOffset14.56mm_Housed_MountingHolesOffset15.98mm -> Connector_Dsub:DSUB-15_Female_Horizontal_P2.77x2.84mm_EdgePinOffset7.70mm_Housed_MountingHolesOffset9.12mm
- RN18, RN19, RN20, RN21: value 10k -> 4K7
- renumbered J3 to J2, J2 to J3
Connections:
- net labels added: EXT_Audio_L, EXT_Audio_R, SCART_Comp, SCART_Switch, Speaker_JAMMA+, Speaker_JAMMA-
- net labels removed: +3V3, -12V, Audio_L, Audio_Mono, Audio_R, BLANK, P1&P2_Shifter_DIR, P1P2_Shifter_DIR, P1_Button1, P1_Button10, P1_Button11, P1_Button12, P1_Button2, P1_Button3, P1_Button4, P1_Button5, P1_Button6, P1_Button7, P1_Button8, P1_Button9, P1_Shifter_DIR, P2_Button1, P2_Button10, P2_Button11, P2_Button12, P2_Button2, P2_Button3, P2_Button4, P2_Button5, P2_Button6, P2_Button7, P2_Button8, P2_Button9, P2_Shifter_DIR, SCART_COMP, SCART_CSYNC, SWITCH, Speaker_L, Speaker_R, VCC
- wire segments 498 -> 241
- no-connect marks 46 -> 43
Other:
- note added: "TO DO LIST:\n- pam8106 audio amp + audio controls\n- Potentiometers for video signal\n- VGA input option (dreamcasts etc.)\n - Also for Dreamcast, and Sync combiner will be necessary\n- THS7375 video amp\n- Button Remapping for software\n- USB"
- note removed: "3V3 I/O to and from Level Shifter"
- note removed: "5V Button Inputs from \nArcade Machine"
- note removed: "Controller Ports & Level Conversion"
- note removed: "Microcontroller"
- note removed: "Player 1"
- note removed: "Player 2"
- note removed: "Slew Rate Control"
- note removed: "Stereo to Mono Combiner"
- note removed: "Sync Stripper"
- note removed: "TO DO LIST:\n- pam8106 audio amp + audio controls\n- BA7046F/LM1881 for Composite Sync\n- Audio mono combiner circuit\n- Potentiometers for video signal\n- VGA input option (dreamcasts etc.)\n - Also for Dreamcast, and Sync combiner will be necessary\n- THS7375 video amp\n- Button Remapping for software"
- note removed: "Video & Audio IN"
- moved on the sheet: J2, J3

Commit message: Schematic mainly done. Working on PCB layout in isolated blocks.
Parts:
- removed D12, D7: LESD3Z5.0CMT1G, Diode_SMD:D_SOD-323, symbol Console2JAMMA:D_TVS_ALT_45deg
- removed RN18, RN19, RN20, RN21, RN22, RN23: 4K7, Resistor_SMD:R_Array_Convex_4x0603, symbol Device:R_Pack04
- added C1: 100n, Capacitor_SMD:C_0603_1608Metric, symbol Device:C
- added C2: 10u, Capacitor_SMD:C_0805_2012Metric, symbol Device:C
- added FID1, FID2: Fiducial, Fiducial:Fiducial_0.5mm_Mask1mm, symbol Mechanical:Fiducial
- added H1, H2, H3, H4: MountingHole_Pad, MountingHole:MountingHole_3.2mm_M3_Pad_Via, symbol Mechanical:MountingHole_Pad
- added J9: USB_B, Connector_USB:USB_B_OST_USB-B1HSxx_Horizontal, symbol Connector:USB_B
- added U1: USBLC6-2P6, Package_TO_SOT_SMD:SOT-666, symbol Power_Protection:USBLC6-2SC6
- added U2: LD1117-3.3, Package_TO_SOT_SMD:TO-252-2, symbol Regulator_Linear:LD1117S33TR_SOT223
- J8: value Conn_01x04 -> Phoenix PTS 1,5/4-5.0
- renumbered D13 to D12, D14 to D13
Connections:
- net EXT_Audio_L is gone; now on net Audio/EXT_Audio_L: J5.1 (IN1)
- net EXT_Audio_R is gone; now on net Audio/EXT_Audio_R: J5.2 (IN2)
- net +5V: now also C1.1, U2.3 (VI)
- net Audio/Speaker_R+: now also J8.1 (Pin_1); no longer J8.3 (Pin_3)
- net Audio/Speaker_R-: now also J8.2 (Pin_2); no longer J8.4 (Pin_4)
- net Digital I/O/P1_1: now also J6.9 (P9)
- net Digital I/O/P1_10: now also J6.6
- net Digital I/O/P1_11: now also J6.14 (P14)
- net Digital I/O/P1_12: now also J6.7
- net Digital I/O/P1_2: now also J6.2
- net Digital I/O/P1_3: now also J6.10 (P10)
- net Digital I/O/P1_4: now also J6.3
- net Digital I/O/P1_5: now also J6.11 (P111)
- net Digital I/O/P1_6: now also J6.4
- net Digital I/O/P1_7: now also J6.12 (P12)
- net Digital I/O/P1_8: now also J6.5
- net Digital I/O/P1_9: now also J6.13 (P13)
- net Digital I/O/P2_1: now also J7.9 (P9)
- net Digital I/O/P2_10: now also J7.6
- net Digital I/O/P2_11: now also J7.14 (P14)
- net Digital I/O/P2_12: now also J7.7
- net Digital I/O/P2_2: now also J7.2
- net Digital I/O/P2_3: now also J7.10 (P10)
- net Digital I/O/P2_4: now also J7.3
- net Digital I/O/P2_5: now also J7.11 (P111)
- net Digital I/O/P2_6: now also J7.4
- net Digital I/O/P2_7: now also J7.12 (P12)
- net Digital I/O/P2_8: now also J7.5
- net Digital I/O/P2_9: now also J7.13 (P13)
- net GND: now also C1.2, C2.2, H1.1, H2.1, H3.1, H4.1, J9.4 (GND), J9.5 (Shield), U1.2 (GND), U2.1 (GND)
- net Speaker_JAMMA+: now also J8.4 (Pin_4); no longer J8.1 (Pin_1)
- net Speaker_JAMMA-: now also J8.3 (Pin_3); no longer J8.2 (Pin_2)
- net SCART_Switch: no longer names the net of J3.8 (P8)
- net VGA_SCK: no longer names the net of J2.15
- net VGA_SDA: no longer names the net of J2.12
- new net: J9.1 (VBUS), U1.5 (VBUS)
- new net: J9.2 (D-), U1.4 (IO2)
- new net: J9.3 (D+), U1.6 (IO1)
- new net +3V3: C2.1, U2.2 (VO)
- new net Digital I/O/USB_D+: U1.1 (IO1)
- new net Digital I/O/USB_D-: U1.3 (IO2)
- no-connect marks 43 -> 46
Other:
- note added: "Digital Audio Controls"
- note added: "Line Level Audio Input"
- note added: "RCA Audio in"
- note added: "TO DO LIST:\n- Potentiometers for video signal?\n- Button Remapping for software\n- Microcontroller VBAT\n- New DB15 Footprint (Standard one is wrong)\n"
- note added: "To External Connector"
- note added: "To JAMMA Edge"
- note removed: "Audio in"
- note removed: "TO DO LIST:\n- pam8106 audio amp + audio controls\n- Potentiometers for video signal\n- VGA input option (dreamcasts etc.)\n - Also for Dreamcast, and Sync combiner will be necessary\n- THS7375 video amp\n- Button Remapping for software\n- USB"
- moved on the sheet: J5, J6, J7, J8
