File: hardware/audio.kicad_sch (KiCad schematic)
At the start: 74 parts, among them U13 PAM8610, U14 PAM8610, U15 74HCT4053, U8 TL072

Commit message: Pushing work I did a few months ago and I forgot to push. Identified some mistakes which I'll fix in a future commit.
Parts:
- removed R24: 10K, Resistor_SMD:R_0603_1608Metric, symbol Device:R
- removed R25: 100K, Resistor_SMD:R_0603_1608Metric, symbol Device:R
- removed U14: PAM8610, Package_DFN_QFN:QFN-40-1EP_6x6mm_P0.5mm_EP4.6x4.6mm, symbol Console2JAMMA:PAM8610
- added R51: 10K, Resistor_SMD:R_0603_1608Metric, symbol Device:R
- added U12: PAM8610, Console2JAMMA:QFN-40-1EP_6x6mm_P0.5mm_EP4.6x4.6mm_ThermalVias, symbol Console2JAMMA:PAM8610
- C83, C84: value 200p -> 10n
- R15, R21, R23: value 10K -> 4K7
- R18: value 4K7 -> 10K
- R22: value 100K -> 4K7
- U13: footprint Package_DFN_QFN:QFN-40-1EP_6x6mm_P0.5mm_EP4.6x4.6mm -> Console2JAMMA:QFN-40-1EP_6x6mm_P0.5mm_EP4.6x4.6mm_ThermalVias
Connections:
- net +3V3 is gone; now on net +5V: R26.2, R47.2
- net +12V: now also U12.12 (PVCCL), U12.19 (PVCCL), U12.26 (AVCC), U12.32 (PVCCR), U12.39 (PVCCR)
- net Audio_L: now also C38.2, U15.4 (Z); no longer C37.2, U15.15 (X)
- net Audio_R: now also C37.2; no longer C38.2
- net EXT_Audio_L: now also U15.3 (Z1); no longer U15.13 (X1)
- net GND: now also R21.2, R22.2, U15.15 (X), U12.11 (PGNDL), U12.20 (PGNDL), U12.24 (AGND), U12.25 (MUTE), U12.28 (AGND), U12.31 (PGNDR), U12.40 (PGNDR), U12.6 (REFGND), U12.7 (AGND1); no longer U15.4 (Z)
- net SCART_Audio_L: now also U15.5 (Z0); no longer U15.12 (X0)
- net Volume: now also U12.5 (VOLUME)
- net ~Mono_Shutdown~: now also U13.29 (~SD~)
- net ~Stereo_Shutdown~: now also U12.29 (~SD~); no longer U13.29 (~SD~)
- net at R16.1, R17.1, R18.2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: now also R51.2
- net at R18.1, R19.2, U8.1: now also R51.1
- net at C42.1: now also U12.1 (RINN); no longer U13.1 (RINN)
- net at C40.1: now also U12.10 (LINN); no longer U13.10 (LINN)
- net at U13.13 (LOUTN), U13.14 (LOUTN): now also C66.2, FB6.1; no longer C51.2, FB2.1
- net at U13.15 (BSLN): now also C66.1; no longer C51.1
- net at C50.2: now also U12.16 (BSLP); no longer U13.16 (BSLP)
- net at C50.1, FB1.1: now also U12.17 (LOUTP), U12.18 (LOUTP); no longer U13.17 (LOUTP), U13.18 (LOUTP)
- net at C41.1: now also U12.2 (RINP); no longer U13.2 (RINP)
- net at C54.2: now also U12.21 (VCLAMPL); no longer U13.21 (VCLAMPL)
- net at U13.22 (COSC): now also C84.1; no longer C83.1
- net at R22.1: now also R15.1, U12.23 (ROSC); no longer U13.23 (ROSC)
- net at C56.2: now also U12.27 (V2P5); no longer U13.27 (V2P5)
- net at U13.3 (AVDD), U13.4 (VREF): now also C82.1; no longer C43.1
- net at C55.2: now also U12.30 (VCLAMPR); no longer U13.30 (VCLAMPR)
- net at C52.1, FB3.1: now also U12.33 (ROUTP), U12.34 (ROUTP); no longer U13.33 (ROUTP), U13.34 (ROUTP)
- net at C52.2: now also U12.35 (BSRP); no longer U13.35 (BSRP)
- net at C53.1: now also U12.36 (BSRN); no longer U13.36 (BSRN)
- net at C53.2, FB4.1: now also U12.37 (ROUTN), U12.38 (ROUTN); no longer U13.37 (ROUTN), U13.38 (ROUTN)
- net at U13.8 (~FADE~): now also R47.1; no longer R26.1
- net at C39.1: now also U12.9 (LINP); no longer U13.9 (LINP)
- net at C81.1: now also U13.1 (RINN)
- net at C79.1: now also U13.10 (LINN)
- net at C64.2: now also U13.16 (BSLP)
- net at C64.1, FB5.1: now also U13.17 (LOUTP), U13.18 (LOUTP)
- net at C80.1: now also U13.2 (RINP)
- net at C67.2: now also U13.21 (VCLAMPL)
- net at C69.2: now also U13.27 (V2P5)
- net at C68.2: now also U13.30 (VCLAMPR)
- net at C87.1: now also U13.33 (ROUTP), U13.34 (ROUTP)
- net at C87.2: now also U13.35 (BSRP)
- net at C88.1: now also U13.36 (BSRN)
- net at C88.2: now also U13.37 (ROUTN), U13.38 (ROUTN)
- net at C78.1: now also U13.9 (LINP)
- net at R23.1: now also R21.1, U13.23 (ROSC)
- new net: C51.1, U12.15 (BSLN)
- new net: C51.2, FB2.1, U12.13 (LOUTN), U12.14 (LOUTN)
- new net: C43.1, U12.3 (AVDD), U12.4 (VREF)
- new net: R26.1, U12.8 (~FADE~)
- new net: C83.1, U12.22 (COSC)
Other:
- note added: "External Stereo Amplifier"
- note added: "JAMMA Mono Amplifier"
- moved on the sheet: C39, C40, C41, C42, C43, C44, C45, C46, C47, C48, C49, C50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
