File: hardware/digital.kicad_sch (KiCad schematic)
At the start: 69 parts, among them J10 Conn_02x03_Odd_Even, J11 Conn_02x05_Odd_Even, J12 Conn_01x03, SW1 SW_Push, SW2 SW_Push, SW3 SW_Push, U10 74LVC4245, U11 74LVC4245, U16 STM32F103VCT6, U9 74LVC4245, Y1 12MHz

Commit message: Pushing work I did a few months ago and I forgot to push. Identified some mistakes which I'll fix in a future commit.
Parts:
- added J13: Conn_01x03, Connector_PinHeader_2.54mm:PinHeader_1x03_P2.54mm_Vertical, symbol Connector_Generic:Conn_01x03
- R46: footprint Resistor_SMD:R_0402_1005Metric -> Resistor_SMD:R_0603_1608Metric
Connections:
- net GND: now also J13.3 (Pin_3)
- net P1_10: now also RN23.2 (R2.1); no longer RN20.2 (R2.1)
- net P1_11: now also RN23.3 (R3.1); no longer RN20.3 (R3.1)
- net P1_12: now also RN23.4 (R4.1); no longer RN20.4 (R4.1)
- net P1_9: now also RN23.1 (R1.1); no longer RN20.1 (R1.1)
- net P2_1: now also RN21.4 (R4.1); no longer RN21.1 (R1.1)
- net P2_10: now also RN22.2 (R2.1); no longer RN23.2 (R2.1)
- net P2_11: now also RN22.3 (R3.1); no longer RN23.3 (R3.1)
- net P2_12: now also RN22.4 (R4.1); no longer RN23.4 (R4.1)
- net P2_2: now also RN21.3 (R3.1); no longer RN21.2 (R2.1)
- net P2_3: now also RN21.2 (R2.1); no longer RN21.3 (R3.1)
- net P2_4: now also RN21.1 (R1.1); no longer RN21.4 (R4.1)
- net P2_5: now also RN20.4 (R4.1); no longer RN22.1 (R1.1)
- net P2_6: now also RN20.3 (R3.1); no longer RN22.2 (R2.1)
- net P2_7: now also RN20.2 (R2.1); no longer RN22.3 (R3.1)
- net P2_8: now also RN20.1 (R1.1); no longer RN22.4 (R4.1)
- net P2_9: now also RN22.1 (R1.1); no longer RN23.1 (R1.1)
- net ~Mono_Shutdown~: now reaches U16.15 (PC0)
- net Audio_Select_~Mono~_Stereo renamed ~Stereo_Shutdown~
- net UART_RX renamed UART_Rx
- net UART_Rx: now also J13.2 (Pin_2)
- net UART_TX renamed UART_Tx
- net UART_Tx: now also J13.1 (Pin_1)
- no-connect marks 7 -> 6
Other:
- note added: "UART Debug & Programming Header"
- moved on the sheet: C70, C71, R34, R35, R40, R41, SW2, SW3
